File: electronics/G65SC151_SBC_V000/G65SC151_SBC_V000.kicad_sch (KiCad schematic)
At the start: 15 parts, among them J14 Conn_01x03, J18 Conn_01x03, J24 Conn_01x03, SW4 switch_DPDT

Commit message: WIP schematic and PCB
Parts:
- removed J14, J18, J24: Conn_01x03, Connector_JST:JST_PH_B3B-PH-K_1x03_P2.00mm_Vertical, symbol Connector_Generic:Conn_01x03
- added C2: 2.2uF, SquantorRcl:C_0805+0603, symbol Device:C
- added C3: C_Polarized, SquantorCapacitor:C-050-100-elco, symbol Device:C_Polarized
- added D1, D2, D3, D4, D5, D6, D7, D8: LED, SquantorDiodes:LED_0603_hand, symbol Device:LED
- added F1: Fuse, Fuse:Fuse_BelFuse_0ZRE0012FF_L8.3mm_W3.8mm, symbol Device:Fuse
- added J1: Jack-DC, SquantorConnectors:BarrelJack_Horizontal_Holed, symbol Connector:Jack-DC
- added J2: VSS, SquantorConnectors:Header-0254-1X08-H010, symbol Connector_Generic:Conn_01x08
- added J3: PORT_A, SquantorConnectors:Header-0254-1X08-H010, symbol Connector_Generic:Conn_01x08
- added J4: LED, SquantorConnectors:Header-0254-1X08-H010, symbol Connector_Generic:Conn_01x08
- added R10, R11, R2, R3, R4, R7, R8, R9: 4.7K, SquantorResistor:R_0603_hand, symbol Device:R
- added U1: ~, Package_LCC:PLCC-68_THT-Socket, symbol Squantor65XX:G65SC151
Connections:
- net GND is gone; now on net VSS: C1.2, R1.2
- net at SW4.4 (SW2_P2): now also F1.1
- net at SW4.5 (SW2_C1): now also J1.1
- net LED: now reaches R5.2
- net LED: now also U1.53 (PD0)
- net VSS: now reaches LED1.2 (C)
- net VSS: now also SW4.3 (SW1_P2), C2.1, C3.2, J2.1 (Pin_1), J2.2 (Pin_2), J2.3 (Pin_3), J2.4 (Pin_4), J2.5 (Pin_5), J2.6 (Pin_6), J2.7 (Pin_7), J2.8 (Pin_8), U1.18 (VSS)
- net VDD: now reaches R6.2
- net VDD: now also C2.2, C3.1, D1.2 (A), D2.2 (A), D3.2 (A), D4.2 (A), D5.2 (A), D6.2 (A), D7.2 (A), D8.2 (A), F1.2, U1.54 (VDD), U1.59 (Vreg)
- net at SW4.2 (SW1_C1): now also J1.2
- new net: D2.1 (K), R3.1
- new net: J4.2 (Pin_2), R3.2
- new net: D5.1 (K), R8.1
- new net: J4.5 (Pin_5), R8.2
- new net: D3.1 (K), R4.1
- new net: D4.1 (K), R7.1
- new net: D6.1 (K), R9.1
- new net: J4.6 (Pin_6), R9.2
- new net: D1.1 (K), R2.1
- new net: J4.1 (Pin_1), R2.2
- new net: J4.3 (Pin_3), R4.2
- new net: J4.4 (Pin_4), R7.2
- new net: J4.7 (Pin_7), R10.2
- new net: J4.8 (Pin_8), R11.2
- new net: D8.1 (K), R11.1
- new net: D7.1 (K), R10.1
- new net CE_ROM: U1.52 (EXTR/PD1)
- new net CLK: U1.63 (CLK)
- new net PA0: J3.1 (Pin_1), U1.42 (PA0)
- new net PA1: J3.2 (Pin_2), U1.41 (PA1)
- new net PA2: J3.3 (Pin_3), U1.40 (PA2)
- new net PA3: J3.4 (Pin_4), U1.39 (PA3)
- new net PA4: J3.5 (Pin_5), U1.38 (PA4)
- new net PA5: J3.6 (Pin_6), U1.37 (PA5)
- new net PA6: J3.7 (Pin_7), U1.36 (PA6)
- new net PA7: J3.8 (Pin_8), U1.35 (PA7)
- new net PB0: U1.50 (PB0)
- new net PB1: U1.49 (PB1)
- new net PB2: U1.48 (PB2)
- new net PB3: U1.47 (PB3)
- new net PB4: U1.46 (PB4)
- new net PB5: U1.45 (PB5)
- new net PB6: U1.44 (PB6)
- new net PB7: U1.43 (PB7)
- new net PC0: U1.27 (PC7)
- new net PC1: U1.28 (PC6)
- new net PC2: U1.29 (PC5)
- new net PC3: U1.30 (PC4)
- new net PC4: U1.31 (PC3)
- new net PC5: U1.32 (PC2)
- new net PC6: U1.33 (PC1)
- new net PC7: U1.34 (PC0)
- new net PD2: U1.51 (PD2)
- no-connect marks 0 -> 2
Other:
- note added: "G65SC151"
- note added: "powersupply"
- note removed: "Interface"
- moved on the sheet: LED1, R5, R6, SW4
